Commit message: Controller Works/need to shrink table height

File: Airhockey/bin/resources/model/panda/panda_arm.urdf (robot description, URDF)
Before this commit: robot panda, 8 links, 7 joints
Links:
- link link0: geometry collision mesh filename=./meshes/collision/link0.obj; visual mesh filename=meshes/visual/link0.obj
- link link1: geometry collision mesh filename=./meshes/collision/link1.obj; visual mesh filename=meshes/visual/link1.obj
- link link2: geometry collision mesh filename=./meshes/collision/link2.obj; visual mesh filename=meshes/visual/link2.obj
- link link3: geometry collision mesh filename=./meshes/collision/link3.obj; visual mesh filename=meshes/visual/link3.obj
- link link4: geometry collision mesh filename=./meshes/collision/link4.obj; visual mesh filename=meshes/visual/link4.obj
- link link5: geometry collision mesh filename=./meshes/collision/link5.obj; visual mesh filename=meshes/visual/link5.obj
- link link6: geometry collision mesh filename=./meshes/collision/link6.obj; visual mesh filename=meshes/visual/link6.obj
- link link7: geometry collision mesh filename=./meshes/collision/link7.obj; visual mesh filename=meshes/visual/link7.obj

Commit message: added mallet to end-effector (control position in controller not adjust yet)

File: Airhockey/bin/resources/model/panda/panda_arm.urdf (robot description, URDF)
Before this commit: robot panda, 8 links, 7 joints
Links:
- link link7: geometry collision cylinder length=0.09 radius=0.055; visual mesh filename=meshes/visual/link7.obj
